File: UINIO-Logic-24MHz.kicad_sch (KiCad schematic)
At the start: 34 parts, among them J1 Conn_02x05_Odd_Even, U1 AT24CS64-XHM, U2 ME6211C33M5G-N, U3 CY7C68013A-56LTX, Y1 24MHz

Commit message: Preparing release version 2.0.0.
Parts:
- removed J1: Conn_02x05_Odd_Even, Connector_IDC:IDC-Header_2x05_P2.54mm_Horizontal, symbol Connector_Generic:Conn_02x05_Odd_Even
- removed JP1, JP2: SolderJumper_2_Open, Jumper:SolderJumper-2_P1.3mm_Open_RoundedPad1.0x1.5mm, symbol Jumper:SolderJumper_2_Open
- added D2: Blue LED, LED_SMD:LED_0603_1608Metric, symbol Device:LED
- added J1: Conn_01x10_Male, Connector_PinHeader_2.54mm:PinHeader_1x10_P2.54mm_Vertical, symbol Connector:Conn_01x10_Male
- added R10, R11, R12, R13, R14, R15, R16, R9: 100K, Resistor_SMD:R_0402_1005Metric, symbol Device:R
- added R18: 10K, Resistor_SMD:R_0402_1005Metric, symbol Device:R
- added U2: 74HC245C, Uinio:TSSOP-20_L6.5-W4.4-P0.65-LS6.4-BL, symbol Uinio:74HC245C
- renumbered D2 to D3, R9 to R17, R10 to R19, R11 to R20, R12 to R21, R13 to R22, R14 to R23, U2 to U3, U3 to U4
Connections:
- net +3.3V: now also R10.1, R11.1, R12.1, R13.1, R14.1, R15.1, R16.1, R9.1, U2.20 (VCC)
- net GND: now also U1.1 (A0), D2.1 (K), J1.1 (Pin_1), J1.10 (Pin_10), U2.1 (DIR), U2.10 (GND), U2.19 (/OE)
- net PB0: now also U2.9 (A8); no longer R1.2
- net PB1: now also U2.8 (A7); no longer R2.2
- net PB2: now also U2.7 (A6); no longer R3.2
- net PB3: now also U2.6 (A5); no longer R4.2
- net PB4: now also U2.5 (A4); no longer R5.2
- net PB5: now also U2.4 (A3); no longer R6.2
- net PB6: now also U2.3 (A2); no longer R7.2
- net PB7: now also U2.2 (A1); no longer R8.2
- net INPUT6: now reaches R3.1
- net INPUT6: now also R14.2, U2.13 (B6)
- net at U4.33 (PA0/~{INT0}): now also R18.2
- net INPUT7: now reaches R2.1
- net INPUT7: now also R15.2, U2.12 (B7)
- net INPUT5: now reaches R4.1
- net INPUT5: now also R13.2, U2.14 (B5)
- net INPUT1: now reaches R8.1
- net INPUT1: now also R9.2, U2.18 (B1)
- net INPUT2: now reaches R7.1
- net INPUT2: now also R10.2, U2.17 (B2)
- net INPUT4: now reaches R5.1
- net INPUT4: now also R12.2, U2.15 (B4)
- net INPUT3: now reaches R6.1
- net INPUT3: now also R11.2, U2.16 (B3)
- net INPUT8: now reaches R1.1
- net INPUT8: now also R16.2, U2.11 (B8)
- new net: J1.6 (Pin_6), R4.2
- new net: J1.8 (Pin_8), R2.2
- new net: D2.2 (A), R18.1
- new net: J1.5 (Pin_5), R5.2
- new net: J1.7 (Pin_7), R3.2
- new net: J1.4 (Pin_4), R6.2
- new net: J1.2 (Pin_2), R8.2
- new net: J1.3 (Pin_3), R7.2
- new net: J1.9 (Pin_9), R1.2
- no-connect marks 27 -> 26
Other:
- note added: "上拉电阻"
- note added: "信 号 收 发 电 路"
- note removed: "牛角座排线接口"
- moved on the sheet: C3, C4, C5, C6, C7, D3, R19, U1

Commit message: Release UINIO-Logic-24MHz version 2.0.0.
Other:
- note added: "信 号 收 发 器"
- note removed: "信 号 收 发 电 路"
Changed lines of the file:
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@@
   (title_block
     (title "UINIO-Logic-24MHz")
-    (date "2022-12-28")
-    (rev "Version 1.0.0")
+    (date "2023-01-29")
+    (rev "Version 2.0.0")
     (company "电子技术博客 UinIO.com")
   )
@@
     (effects (font (size 3 3)) (justify left bottom))
   )
-  (text "信\n号\n收\n发\n电\n路" (at 33.02 54.61 0)
+  (text "信\n号\n收\n发\n器" (at 34.29 52.07 0)
     (effects (font (size 3 3)) (justify left bottom))
   )

Commit message: Prepare UINIO-Logic-24MHz version 3.0.0.
Parts:
- added R24, R25: 5.1K, Resistor_SMD:R_0402_1005Metric, symbol Device:R
Connections:
- net GND: now also R24.2, R25.2
- net at USB1.A5 (CC1): now also R24.1
- net at USB1.A8 (SBU1): now also R25.1
- no-connect marks 26 -> 24
Other:
- moved on the sheet: USB1
