File: UINIO-Logic-24MHz.kicad_sch (KiCad schematic)
At the start: 51 parts, among them J1 Conn_01x10_Pin, U1 AT24CS64-XHM, U2 74HC245C, U3 ME6211C33M5G-N, U4 CY7C68013A-56LTX, Y1 24MHz

Commit message: Release UINIO-Logic-24MHz version 5.0.0.
Parts:
- D4: footprint Diode_SMD:D_SMA -> Diode_SMD:Nexperia_CFP3_SOD-123W
Changed lines of the file:
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@@
 			)
 		)
-		(property "Footprint" "Diode_SMD:D_SMA"
+		(property "Footprint" "Diode_SMD:Nexperia_CFP3_SOD-123W"
 			(at 154.94 131.445 0)
 			(effects

Commit message: Release UINIO-Logic-24MHz version 5.0.0.
Parts:
- C1, C2: footprint Capacitor_SMD:C_0402_1005Metric -> Capacitor_SMD:C_0603_1608Metric
Changed lines of the file:
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@@
 			)
 		)
-		(property "Footprint" "Capacitor_SMD:C_0402_1005Metric"
+		(property "Footprint" "Capacitor_SMD:C_0603_1608Metric"
 			(at 152.0952 153.67 0)
 			(effects
@@
 			)
 		)
-		(property "Footprint" "Capacitor_SMD:C_0402_1005Metric"
+		(property "Footprint" "Capacitor_SMD:C_0603_1608Metric"
 			(at 113.9952 153.67 0)
 			(effects

Commit message: Release UINIO-Logic-24MHz version 5.0.0.
Parts:
- R17: footprint Resistor_SMD:R_0603_1608Metric -> Resistor_SMD:R_0402_1005Metric
Changed lines of the file:
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@@
 			)
 		)
-		(property "Footprint" "Resistor_SMD:R_0603_1608Metric"
+		(property "Footprint" "Resistor_SMD:R_0402_1005Metric"
 			(at 164.338 161.29 90)
 			(effects
