File: UINIO-Logic-24MHz.kicad_pcb (KiCad board)
At the start: 2 copper layers, 48.8 x 25.5 mm, 49 parts, among them J1 Conn_01x10_Male, U1 AT24CS64-XHM, U2 74HC245C, U3 ME6211C33M5G-N, U4 CY7C68013A-56LTX, Y1 24MHz

Commit message: Release UINIO-Logic-24MHz version 2.0.0.
Parts:
- moved ? 0.32 mm to (144.7, 118.6)
Routing:
- net Net-(J1-Pad6): track 6.35 -> 5.64 mm
- net Net-(C8-Pad2): track 22.5 -> 21.8 mm
- net /PB5: track 6.83 -> 6.13 mm
- net /PB0: track 6.96 -> 6.27 mm
- net /PB7: track 6.96 -> 6.27 mm
- net /PB6: track 6.90 -> 6.22 mm
- net /PB2: track 6.83 -> 6.17 mm
- net /PB1: track 6.90 -> 6.24 mm
- net GND: track 77.9 -> 77.8 mm, vias 11 -> 13

Commit message: Prepare UINIO-Logic-24MHz version 3.0.0.
Parts:
- added R24: 5.1K, Resistor_SMD:R_0402_1005Metric, F.Cu at (148.8, 128.5)
- added R25: 5.1K, Resistor_SMD:R_0402_1005Metric, F.Cu at (145.7, 109.1)
- moved D1 0.58 mm to (148.5, 109.7)
- moved R17 0.58 mm to (146.9, 109.1)
- moved C8 0.34 mm to (142.3, 128.5)
- moved Y1 0.34 mm to (144.8, 127.3)
- moved C9 0.34 mm to (147.4, 128.5)
- moved U1 0.17 mm to (128.7, 109.6)
Connections:
- USB1 pad A5: unconnected-(USB1-PadA5) -> Net-(USB1-PadA5)
- USB1 pad A8: unconnected-(USB1-PadA8) -> Net-(USB1-PadA8)
Routing:
- net Net-(USB1-PadA5): track 0.00 -> 9.66 mm, vias 0 -> 2
- net Net-(USB1-PadA8): track 0.00 -> 9.40 mm, vias 0 -> 2
- net GND: track 77.8 -> 84.8 mm, vias 13 -> 14
- net +3.3V: track 166.1 -> 167.1 mm
- net Net-(C9-Pad2): track 23.7 -> 24.4 mm
Other:
- board text added: "8通道 24MHz采样频率"
- board text removed: "24MHz 采样频率"
- board text removed: "8 个采样通道"

Commit message: Prepare UINIO-Logic-24MHz version 3.0.0.
Parts:
- moved C8 0.25 mm to (142.0, 128.5)
- moved C9 0.25 mm to (147.2, 128.5)
- moved Y1 0.25 mm to (144.6, 127.3)
Routing:
- net GND: track 84.8 -> 82.7 mm, vias 14 -> 15
- net +3.3V: track 167.1 -> 166.4 mm
Other:
- board text added: "Version 3.0.0"
- board text removed: "Version 2.0.0"

Commit message: Prepare UINIO-Logic-24MHz version 3.0.0.
Parts:
- moved ? 0.12 mm to (144.7, 118.7)

Commit message: Release UINIO-Logic-24MHz version 3.0.0.
Parts:
- D1: value Red LED -> LED Red
- D2: value Blue LED -> LED Yellow
- D3: value Blue LED -> LED Green
Routing:
- net GND: track 82.7 -> 104.6 mm, vias 15 -> 23
Other:
- board text added: "CH0"
- board text removed: "CH8"

Commit message: Prepare version 3.1.0.
Parts:
- removed the ? at (144.7, 118.7)
- removed the ? at (130.6, 118.6)
- added ?: LOGO, LOGO, B.Cu at (136.1, 118.8)
- added ?: LOGO, LOGO, B.Cu at (120.4, 118.8)
- J1: value Conn_01x10_Male -> Conn_01x10_Pin
- moved HOLE1 0.41 mm to (114.5, 108.7)
- moved HOLE2 0.41 mm to (114.5, 128.7)
- moved USB1 0.18 mm to (150.6, 118.8)
Other:
- board text added: "UinIO.com"
- board text added: "Version 3.1.0"
- board text removed: "Version 3.0.0"

Commit message: Release UINIO-Logic-24MHz version 3.1.0.
Parts:
- moved C1 24.9 mm to (165.0, 97.2)
- moved C10 24.9 mm to (161.6, 115.4)
- moved C8 24.9 mm to (163.2, 115.4)
- moved D1 24.9 mm to (169.7, 96.6)
- moved HOLE3 24.9 mm to (173.4, 95.6)
- moved R21 24.9 mm to (150.7, 99.3)
- moved R24 24.9 mm to (170.0, 115.4)
- moved U3 24.9 mm to (162.4, 96.7)
- moved Y1 24.9 mm to (165.8, 114.3)
- moved D3 24.9 mm to (156.3, 114.9)
- moved HOLE4 24.9 mm to (173.4, 115.6)
- moved R11 24.9 mm to (142.6, 115.5)
- moved R18 24.9 mm to (151.0, 115.2)
- moved R19 24.9 mm to (154.7, 115.2)
- moved R23 24.9 mm to (160.3, 115.4)
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Other:
- outline, holes or cut-outs redrawn
