File: UINIO-Logic-24MHz.kicad_pcb (KiCad board)
At the start: 2 copper layers, 52 x 25.4 mm, 55 parts, among them J1 Conn_01x10_Pin, U1 AT24CS64-XHM, U2 74HC245C, U3 ME6211C33M5G-N, U4 CY7C68013A-56LTX, Y1 24MHz

Commit message: Release UINIO-Logic-24MHz version 5.0.0.
Parts:
- C1, C2: footprint Capacitor_SMD:C_0402_1005Metric -> Capacitor_SMD:C_0603_1608Metric
- moved Y1 1.04 mm to (138.3, 96.6)
- moved C8 0.95 mm to (139.3, 99.1)
- moved C9 0.95 mm to (137.2, 99.1)
- moved C12 0.61 mm to (139.9, 110.8)
- moved C7 0.61 mm to (139.4, 107.8)
- moved R20 0.61 mm to (139.4, 102.8)
- moved R24 0.52 mm to (134.7, 101.3)
- moved D5 0.52 mm to (133.9, 106.8)
- moved D6 0.52 mm to (133.9, 104.3)
- moved R25 0.52 mm to (134.7, 109.9)
- moved C2 0.30 mm to (143.0, 115.3)
- moved C1 0.30 mm to (137.3, 115.3)
Routing:
- net +3.3V: track 170.1 -> 167.3 mm
- net Net-(U4-XTALIN): track 25.1 -> 24.1 mm
- net Net-(U4-XTALOUT): track 20.3 -> 19.2 mm
- net Net-(U4-WAKEUP): track 2.79 -> 2.18 mm
- net GND: track 24.1 -> 24.0 mm, vias 33 -> 34

Commit message: Release UINIO-Logic-24MHz version 5.0.0.
Parts:
- R17: footprint Resistor_SMD:R_0603_1608Metric -> Resistor_SMD:R_0402_1005Metric
- moved C10 3.46 mm to (142.1, 98.7)
- moved R23 3.41 mm to (143.6, 98.6)
- moved R17 0.32 mm to (132.2, 115.9)
- moved C8 0.09 mm to (139.3, 99.1)
- moved C9 0.09 mm to (137.3, 99.1)
Routing:
- net Net-(U4-~{RESET}): track 7.47 -> 4.05 mm
- net GND: vias 34 -> 59
